File: WISP_display_board.kicad_sch (KiCad schematic)
At the start: 109 parts, among them J1 Conn_01x09_Socket, U1 74HC595, U2 74HC595, U3 74HC595, U4 74HC595, U6 74HC595, U7 74HC595, U8 74HC595, U9 74HC595

Commit message: Full 15 rough draft
Parts:
- removed J1: Conn_01x09_Socket, Connector_PinSocket_2.54mm:PinSocket_1x09_P2.54mm_Vertical, symbol Connector:Conn_01x09_Socket
- added Brd3, Brd4, Brd5, Brd6, Brd7, Brd8: SSD1306, ssd1306_custom:128x64OLED, symbol ssd1306_custom:SSD1306
- added J1: Conn_01x10_Socket, Connector_PinHeader_2.54mm:PinHeader_1x10_P2.54mm_Vertical, symbol Connector:Conn_01x10_Socket
- added R61, R62, R63, R64, R65, R66, R67, R68, R69, R70, R71, R72, R73, R74, R75, R76: 4.7k, Resistor_SMD:R_0805_2012Metric_Pad1.20x1.40mm_HandSolder, symbol Device:R_Small
- added U5: TCA9548APWR, Package_SO:TSSOP-24_4.4x7.8mm_P0.65mm, symbol Interface_Expansion:TCA9548APWR
Connections:
- net +3.3V: now also Brd3.2 (VCC), Brd4.2 (VCC), Brd5.2 (VCC), Brd6.2 (VCC), Brd7.2 (VCC), Brd8.2 (VCC), J1.10 (Pin_10), R61.1, R62.2, R63.2, R64.1, R65.2, R66.1, R67.2, R68.1, R69.2, R70.1, R71.2, R72.1, R73.2, R74.1, R75.2, R76.1, U5.24 (VCC), U5.3 (~{RESET})
- net GND: now also Brd3.1 (GND), Brd4.1 (GND), Brd5.1 (GND), Brd6.1 (GND), Brd7.1 (GND), Brd8.1 (GND), J1.9 (Pin_9), U5.12 (GND)
- net I2C1_SCL: now also J1.4 (Pin_4), U5.22 (SCL); no longer Brd1.3 (SCL)
- net I2C1_SDA: now also J1.5 (Pin_5), U5.23 (SDA); no longer Brd1.4 (SDA)
- net SPI3_MOSI: now also J1.3 (Pin_3)
- net SPI3_SCK: now also J1.2 (Pin_2)
- net SPI3_STCP: now also J1.1 (Pin_1)
- net I2C3_SCL renamed SC1
- net SC1: now also R64.2, U5.7 (SC1)
- net I2C3_SDA renamed SD1
- net SD1: now also R63.1, U5.6 (SD1)
- new net I2C_A0: J1.6 (Pin_6), U5.1 (A0)
- new net I2C_A1: J1.7 (Pin_7), U5.2 (A1)
- new net I2C_A2: J1.8 (Pin_8), U5.21 (A2)
- new net SC0: Brd1.3 (SCL), R61.2, U5.5 (SC0)
- new net SC2: Brd3.3 (SCL), R66.2, U5.9 (SC2)
- new net SC3: Brd4.3 (SCL), R68.2, U5.11 (SC3)
- new net SC4: Brd5.3 (SCL), R70.2, U5.14 (SC4)
- new net SC5: Brd6.3 (SCL), R72.2, U5.16 (SC5)
- new net SC6: Brd7.3 (SCL), R74.2, U5.18 (SC6)
- new net SC7: Brd8.3 (SCL), R76.2, U5.20 (SC7)
- new net SD0: Brd1.4 (SDA), R62.1, U5.4 (SD0)
- new net SD2: Brd3.4 (SDA), R65.1, U5.8 (SD2)
- new net SD3: Brd4.4 (SDA), R67.1, U5.10 (SD3)
- new net SD4: Brd5.4 (SDA), R69.1, U5.13 (SD4)
- new net SD5: Brd6.4 (SDA), R71.1, U5.15 (SD5)
- new net SD6: Brd7.4 (SDA), R73.1, U5.17 (SD6)
- new net SD7: Brd8.4 (SDA), R75.1, U5.19 (SD7)
Other:
- note added: "TEST-BOARD"
- note removed: "Test-Board"
- company: (none) -> Wisconsin Space Program
- title: (none) -> P&ID Display Board
- moved on the sheet: Brd1, C1, C2, C3, C4, C5, C6, C7, C8, D1, D10, D11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

Commit message: V1 routing
Parts:
- removed C6, C7, C8: 0.1uF, Capacitor_SMD:C_0603_1608Metric_Pad1.08x0.95mm_HandSolder, symbol Device:C_Small
- removed D21, D22, D23, D24, D25, D26, D27, D28, D29, D30: LED_Dual_AAKK, LED_SMD:LED_Kingbright_KPBD-3224, symbol Device:LED_Dual_AAKK
- removed R41, R42, R43, R44, R45, R46, R47, R48, R49, R50, R51, R52, R53, R54, R55, R56, R57, R58, R59, R60: 750, Resistor_SMD:R_0805_2012Metric_Pad1.20x1.40mm_HandSolder, symbol Device:R
- removed U2, U3, U4: 74HC595, Package_SO:SOIC-16W_7.5x12.8mm_P1.27mm, symbol 74xx:74HC595
- J1: footprint Connector_PinHeader_2.54mm:PinHeader_1x10_P2.54mm_Vertical -> Connector_JST:JST_XH_B10B-XH-A_1x10_P2.50mm_Vertical
- renumbered R9 to R10, R10 to R11, R11 to R12, R12 to R13, R13 to R14, R14 to R15, R15 to R16, R62 to R17, R63 to R18, R65 to R19, R32 to R2, R67 to R20, R61 to R21, R64 to R22, R66 to R23, R68 to R24, R16 to R25, R17 to R26, R18 to R27, R19 to R28, R20 to R29, R2 to R3, R21 to R30, R22 to R31, R23 to R32, R24 to R33, R25 to R34, R26 to R35, R27 to R36, R28 to R37, R29 to R38, R30 to R39, R3 to R4, R31 to R40, R69 to R41, R71 to R42, R73 to R43, R75 to R44, R70 to R45, R72 to R46, R74 to R47, R76 to R48, R33 to R49, R4 to R5, R34 to R50, R35 to R51, R36 to R52, R37 to R53, R38 to R54, R39 to R55, R40 to R56, R5 to R6, R6 to R7, R7 to R8, R8 to R9, U5 to U1, U6 to U2, U7 to U3, U8 to U4, U9 to U5, U1 to U6
Connections:
- net +3.3V: now also J1.1 (Pin_1); no longer J1.10 (Pin_10)
- net GND: now also J1.2 (Pin_2); no longer J1.9 (Pin_9)
- net I2C1_SCL: now also J1.7 (Pin_7); no longer J1.4 (Pin_4)
- net I2C1_SDA: now also J1.6 (Pin_6); no longer J1.5 (Pin_5)
- net I2C_A0: now also J1.5 (Pin_5); no longer J1.6 (Pin_6)
- net I2C_A1: now also J1.4 (Pin_4); no longer J1.7 (Pin_7)
- net I2C_A2: now also J1.3 (Pin_3); no longer J1.8 (Pin_8)
- net SPI3_MOSI: now also J1.8 (Pin_8); no longer J1.3 (Pin_3)
- net SPI3_SCK: now also J1.9 (Pin_9); no longer J1.2 (Pin_2)
- net SPI3_STCP: now also J1.10 (Pin_10); no longer J1.1 (Pin_1)
- no-connect marks 5 -> 0

Commit message: Rough draft V2
Parts:
- C1, C2, C3, C4, C5: footprint Capacitor_SMD:C_0603_1608Metric_Pad1.08x0.95mm_HandSolder -> Capacitor_SMD:C_0805_2012Metric_Pad1.18x1.45mm_HandSolder
- J1: footprint Connector_JST:JST_XH_B10B-XH-A_1x10_P2.50mm_Vertical -> Connector_PinSocket_2.54mm:PinSocket_1x10_P2.54mm_Vertical
Other:
- moved on the sheet: C1, C2, C3, C4, C5, U2, U3, U4, U5, U6

Commit message: John revisions 9/7
Other:
- note added: "CTRL_CONNECTION"
- note removed: "TEST-BOARD"
Changed lines of the file:
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@@
 		)
 	)
-	(text "TEST-BOARD"
+	(text "CTRL_CONNECTION"
 		(exclude_from_sim no)
-		(at 276.098 175.514 0)
+		(at 250.19 168.91 0)
 		(effects
 			(font
@@
 	(text "SENSORS"
 		(exclude_from_sim no)
-		(at 36.068 170.688 0)
+		(at 33.528 169.164 0)
 		(effects
 			(font

Commit message: Rough Draft V3
Parts:
- removed Brd8: SSD1306, ssd1306_custom:128x64OLED, symbol ssd1306_custom:SSD1306
- removed R44, R48: 4.7k, Resistor_SMD:R_0805_2012Metric_Pad1.20x1.40mm_HandSolder, symbol Device:R_Small
- added H1, H2, H3, H4: MountingHole, MountingHole:MountingHole_3.2mm_M3, symbol Mechanical:MountingHole
Connections:
- net SC7: no longer names the net of U1.20 (SC7)
- net SD7: no longer names the net of U1.19 (SD7)
- no-connect marks 0 -> 2

Commit message: Fixed LED orientation
Parts:
- removed D1, D10, D11, D12, D13, D14, D15, D16, D17, D18, D19, D2, D20, D3, D4, D5, D6, D7, D8, D9: LED_Dual_AAKK, LED_SMD:LED_Kingbright_KPBD-3224, symbol Device:LED_Dual_AAKK
- added D1, D10, D11, D12, D13, D14, D15, D16, D17, D18, D19, D2, D20, D3, D4, D5, D6, D7, D8, D9: LED_Dual_AKAK, LED_SMD:LED_Kingbright_KPBD-3224, symbol Device:LED_Dual_AKAK
Connections:
- net GND: now also D1.2 (K1), D1.4 (K2), D10.2 (K1), D10.4 (K2), D11.2 (K1), D11.4 (K2), D12.2 (K1), D12.4 (K2), D13.2 (K1), D13.4 (K2), D14.2 (K1), D14.4 (K2), D15.2 (K1), D15.4 (K2), D16.2 (K1), D16.4 (K2), D17.2 (K1), D17.4 (K2), D18.2 (K1), D18.4 (K2), D19.2 (K1), D19.4 (K2), D2.2 (K1), D2.4 (K2), D20.2 (K1), D20.4 (K2), D3.2 (K1), D3.4 (K2), D4.2 (K1), D4.4 (K2), D5.2 (K1), D5.4 (K2), D6.2 (K1), D6.4 (K2), D7.2 (K1), D7.4 (K2), D8.2 (K1), D8.4 (K2), D9.2 (K1), D9.4 (K2)
- net at R56.2: now also D20.3 (A2)
- net at R1.2: now also D1.1 (A1)
- net at R2.2: now also D1.3 (A2)
- net at R27.2: now also D10.1 (A1)
- net at R34.2: now also D13.3 (A2)
- net at R9.2: now also D5.1 (A1)
- net at R10.2: now also D5.3 (A2)
- net at R32.2: now also D12.3 (A2)
- net at R4.2: now also D2.3 (A2)
- net at R3.2: now also D2.1 (A1)
- net at R50.2: now also D17.3 (A2)
- net at R28.2: now also D10.3 (A2)
- net at R13.2: now also D7.1 (A1)
- net at R6.2: now also D3.3 (A2)
- net at R53.2: now also D19.1 (A1)
- net at R54.2: now also D19.3 (A2)
- net at R30.2: now also D11.3 (A2)
- net at R25.2: now also D9.1 (A1)
- net at R26.2: now also D9.3 (A2)
- net at R49.2: now also D17.1 (A1)
- net at R29.2: now also D11.1 (A1)
- net at R11.2: now also D6.1 (A1)
- net at R12.2: now also D6.3 (A2)
- net at R39.2: now also D16.1 (A1)
- net at R40.2: now also D16.3 (A2)
- net at R52.2: now also D18.3 (A2)
- net at R33.2: now also D13.1 (A1)
- net at R14.2: now also D7.3 (A2)
- net at R7.2: now also D4.1 (A1)
- net at R8.2: now also D4.3 (A2)
- net at R31.2: now also D12.1 (A1)
- net at R5.2: now also D3.1 (A1)
- net at R15.2: now also D8.1 (A1)
- net at R16.2: now also D8.3 (A2)
- net at R38.2: now also D15.3 (A2)
- net at R51.2: now also D18.1 (A1)
- net at R37.2: now also D15.1 (A1)
- net at R35.2: now also D14.1 (A1)
- net at R55.2: now also D20.1 (A1)
- net at R36.2: now also D14.3 (A2)

Commit message: Adam revisions 10/6
Connections:
- net SER_OUT5: no longer names the net of U6.9 (QH')
- no-connect marks 2 -> 3
Changed lines of the file:
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@@
+	)
+	(no_connect
+		(at 311.15 64.77)
 	)
 	(no_connect
@@
 		)
 	)
-	(label "SER_OUT5"
-		(at 311.15 64.77 0)
-		(effects
-			(font
-				(size 1.27 1.27)
-			)
-			(justify left bottom)
-		)
-	)
