File: WISP_display_board.kicad_pcb (KiCad board)
At the start: 4 copper layers, 220 x 160 mm, 97 parts, among them J1 Conn_01x10_Socket, U1 TCA9548APWR, U2 74HC595, U3 74HC595, U4 74HC595, U5 74HC595, U6 74HC595

Commit message: Adam revisions 10/6
Parts:
- Brd1, Brd2, Brd3, Brd4, Brd5, Brd6, Brd7: footprint ssd1306_custom:128x64OLED -> ssd1306_custom:ssd1306_custom_edited
- moved C1 151.4 mm to (199.2, 185.2)
- moved R1 151.4 mm to (187.7, 187.7)
- moved R2 151.4 mm to (187.7, 191.2)
- moved R3 151.4 mm to (187.7, 194.7)
- moved R4 151.4 mm to (187.7, 198.2)
- moved R5 151.4 mm to (209.2, 198.2)
- moved R7 151.4 mm to (209.2, 191.2)
- moved R8 151.4 mm to (209.2, 187.7)
- moved U2 151.4 mm to (198.2, 193.2)
- moved R6 151.4 mm to (209.2, 194.7)
- moved D17 142.1 mm to (286.9, 73.1)
- moved D18 130.3 mm to (287.1, 79.8)
- moved D3 123.1 mm to (194.7, 157.9)
- moved D4 111.1 mm to (205.0, 158.0)
- moved C4 110.8 mm to (234.7, 185.0)
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Connections:
- U6 pad 9: /SER_OUT5 -> unconnected-(U6-QH&apos;-Pad9)
Routing:
- net /SPI3_SCK: track 466.0 -> 184.6 mm, vias 8 -> 5
- net /SPI3_STCP: track 461.8 -> 181.2 mm, vias 8 -> 5
- net +3.3V: track 303.3 -> 110.4 mm, vias 12 -> 2
- net /SPI3_MOSI: track 189.4 -> 37.8 mm, vias 2 -> 1
- net Net-(D19-A1): track 127.3 -> 0.00 mm
- net Net-(D19-A2): track 126.4 -> 0.00 mm
- net /SER_OUT3: track 192.3 -> 79.7 mm
- net Net-(D20-A1): track 107.1 -> 0.00 mm
- net /SER_OUT4: track 155.3 -> 50.1 mm
- net Net-(D20-A2): track 105.0 -> 0.00 mm
- net /SER_OUT2: track 137.0 -> 43.9 mm
- net Net-(D17-A2): track 87.0 -> 0.00 mm
- net Net-(D17-A1): track 84.6 -> 0.00 mm
- net Net-(D18-A2): track 76.4 -> 0.00 mm
- net Net-(D18-A1): track 74.6 -> 0.00 mm
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
Commit message: Rough draft V4
Parts:
- moved R20 4.19 mm to (266.0, 69.5)
- moved R24 4.19 mm to (260.5, 69.5)
- moved R18 4.19 mm to (350.0, 110.7)
- moved R22 4.19 mm to (345.5, 110.7)
- moved R17 3.18 mm to (248.3, 143.8)
- moved R21 3.18 mm to (243.3, 143.8)
- moved R19 2.74 mm to (216.5, 89.8)
- moved R23 2.74 mm to (211.5, 89.8)
- moved C5 1.50 mm to (268.5, 184.9)
- moved C3 1.40 mm to (302.8, 185.3)
- moved C4 1.08 mm to (233.7, 185.5)
- moved C1 1.00 mm to (198.2, 185.3)
- moved C2 0.96 mm to (336.1, 185.6)
- moved D10 0.30 mm to (287.3, 150.3)
- moved D20 0.20 mm to (286.9, 112.5)
Routing:
- net Net-(D7-A1): track 0.00 -> 175.8 mm
- net +3.3V: track 110.4 -> 283.9 mm, vias 2 -> 7
- net Net-(D7-A2): track 0.00 -> 171.7 mm
- net Net-(D18-A2): track 0.00 -> 158.5 mm
- net Net-(D8-A1): track 0.00 -> 157.4 mm
- net Net-(D8-A2): track 0.00 -> 152.5 mm
- net Net-(D18-A1): track 0.00 -> 152.1 mm
- net Net-(D17-A2): track 0.00 -> 142.5 mm
- net Net-(D17-A1): track 0.00 -> 134.4 mm
- net Net-(D5-A2): track 0.00 -> 108.3 mm
- net Net-(D20-A2): track 0.00 -> 108.1 mm
- net Net-(D20-A1): track 0.00 -> 107.8 mm
- net Net-(D6-A2): track 0.00 -> 107.0 mm
- net Net-(D5-A1): track 0.00 -> 105.5 mm
- net Net-(D6-A1): track 0.00 -> 105.5 mm
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